Commit message: add 7月27号

File: thurobot/urdf/smartcar.urdf (robot description, URDF)
Before this commit: robot smartcar, 6 links, 5 joints
Links:
- removed link base_link
- added link base_footprint; visual box size=0.25 .16 .05
Joints:
- joint left_back_wheel_joint: parent base_link -> base_footprint
- joint left_front_wheel_joint: parent base_link -> base_footprint
- joint right_back_wheel_joint: parent base_link -> base_footprint
- joint right_front_wheel_joint: parent base_link -> base_footprint
- joint tobox: parent base_link -> base_footprint

File: thurobot/xacro/gazebo/thurobot_base_gazebo.xacro (robot description, xacro)
@@ -45,5 +45,5 @@
         <joint name="${prefix}_wheel_joint" type="continuous">
             <origin xyz="0 ${reflect*wheel_joint_y} ${-wheel_joint_z}" rpy="0 0 0"/>
-            <parent link="base_link"/>
+            <parent link="base_footprint"/>
             <child link="${prefix}_wheel_link"/>
             <axis xyz="0 1 0"/>
@@ -84,5 +84,5 @@
         <joint name="${prefix}_caster_joint" type="continuous">
             <origin xyz="${reflect*caster_joint_x} 0 ${-(base_length/2 + caster_radius)}" rpy="0 0 0"/>
-            <parent link="base_link"/>
+            <parent link="base_footprint"/>
             <child link="${prefix}_caster_link"/>
             <axis xyz="0 1 0"/>
@@ -123,7 +123,7 @@
             <origin xyz="0 0 ${base_length/2 + caster_radius*2}" rpy="0 0 0" />
             <parent link="base_footprint"/>
-            <child link="base_link" />
+            <child link="base_footprint" />
         </joint>
-        <link name="base_link">
+        <link name="base_footprint">
             <visual>
                 <origin xyz=" 0 0 0" rpy="0 0 0" />
@@ -141,5 +141,5 @@
             <cylinder_inertial_matrix  m="${base_mass}" r="${base_radius}" h="${base_length}" />
         </link>
-        <gazebo reference="base_link">
+        <gazebo reference="base_footprint">
             <material>Gazebo/Blue</material>
         </gazebo>

File: thurobot/xacro/gazebo/thurobot_with_camera_gazebo.xacro (robot description, xacro)
@@ -9,5 +9,5 @@
     <joint name="camera_joint" type="fixed">
         <origin xyz="${camera_offset_x} ${camera_offset_y} ${camera_offset_z}" rpy="0 0 0" />
-        <parent link="base_link"/>
+        <parent link="base_footprint"/>
         <child link="camera_link"/>
     </joint>

File: thurobot/xacro/gazebo/thurobot_with_kinect_gazebo.xacro (robot description, xacro)
@@ -9,5 +9,5 @@
     <joint name="kinect_joint" type="fixed">
         <origin xyz="${kinect_offset_x} ${kinect_offset_y} ${kinect_offset_z}" rpy="0 0 0" />
-        <parent link="base_link"/>
+        <parent link="base_footprint"/>
         <child link="kinect_link"/>
     </joint>

File: thurobot/xacro/gazebo/thurobot_with_laser_gazebo.xacro (robot description, xacro)
@@ -9,5 +9,5 @@
     <joint name="lidar_joint" type="fixed">
         <origin xyz="${lidar_offset_x} ${lidar_offset_y} ${lidar_offset_z}" rpy="0 0 0" />
-        <parent link="base_link"/>
+        <parent link="base_footprint"/>
         <child link="laser_link"/>
     </joint>

File: thurobot/xacro/thurobot_base.xacro (robot description, xacro)
@@ -25,5 +25,5 @@
         <joint name="${prefix}_wheel_joint" type="continuous">
             <origin xyz="0 ${reflect*wheel_joint_y} ${-wheel_joint_z}" rpy="0 0 0"/>
-            <parent link="base_link"/>
+            <parent link="base_footprint"/>
             <child link="${prefix}_wheel_link"/>
             <axis xyz="0 1 0"/>
@@ -43,5 +43,5 @@
         <joint name="${prefix}_caster_joint" type="continuous">
             <origin xyz="${reflect*caster_joint_x} 0 ${-(base_length/2 + caster_radius)}" rpy="0 0 0"/>
-            <parent link="base_link"/>
+            <parent link="base_footprint"/>
             <child link="${prefix}_caster_link"/>
             <axis xyz="0 1 0"/>
@@ -69,7 +69,7 @@
             <origin xyz="0 0 ${base_length/2 + caster_radius*2}" rpy="0 0 0" />
             <parent link="base_footprint"/>
-            <child link="base_link" />
+            <child link="base_footprint" />
         </joint>
-        <link name="base_link">
+        <link name="base_footprint">
             <visual>
                 <origin xyz=" 0 0 0" rpy="0 0 0" />

File: thurobot/xacro/thurobot_with_camera.xacro (robot description, xacro)
@@ -10,5 +10,5 @@
     <joint name="camera_joint" type="fixed">
         <origin xyz="${camera_offset_x} ${camera_offset_y} ${camera_offset_z}" rpy="0 0 0" />
-        <parent link="base_link"/>
+        <parent link="base_footprint"/>
         <child link="camera_link"/>
     </joint>
